File: ESP32Superexpander.2ndattempt/ESP32wShiftRegisters-v2-bug/ESP32wShiftRegisters.sch (KiCad schematic (older format))
At the start: 32 parts, among them J101 CNT1_in, J102 S1_in, J103 S1_in, J104 CNT2_in, J105 S1_in, J106 S1_in, J107 S1_in, J108 S1_in, J109 S1_in, J110 S1_in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

Commit message: Complete Project
Parts:
- removed H102, H103, H104: MountingHole, MountingHole:MountingHole_3.2mm_M3, symbol Mechanical:MountingHole
- removed J111: Conn_02x12_Odd_Even, Connector_PinHeader_2.54mm:PinHeader_2x12_P2.54mm_Vertical, symbol Connector_Generic:Conn_02x12_Odd_Even
- removed J123, J124: Conn_02x02_Odd_Even, Connector_PinHeader_2.54mm:PinHeader_2x02_P2.54mm_Vertical, symbol Connector_Generic:Conn_02x02_Odd_Even
- removed U104: CRE1S0505S3C, LM2596Module:LM2596_Module, symbol Regulator_Switching:CRE1S0505S3C
- added C101: 100uF, Capacitor_THT:CP_Radial_Tantal_D5.5mm_P5.00mm, symbol Device:CP
- added D101: DIODE, Diode_THT:D_5KP_P10.16mm_Horizontal, symbol pspice:DIODE
- added H102, H103, H104: MountingHole_Pad, MountingHole:MountingHole_3.2mm_M3, symbol ESP32wShiftRegisters-rescue:MountingHole_Pad-Mechanical
- added J111: EN VP VN 34 35 32 33 25, Connector_PinSocket_2.54mm:PinSocket_1x08_P2.54mm_Vertical, symbol Connector:Conn_01x08_Female
- added U104: L7805, Package_TO_SOT_THT:TO-220-3_Vertical, symbol Regulator_Linear:L7805
- H101: footprint MountingHole:MountingHole_3.2mm_M3_Pad_Via -> MountingHole:MountingHole_3.2mm_M3
Connections:
- net labels added: 3VP2S_SCK, 3VP2S_SDA, 3VS2P_SCL, 3VS2P_SDA, P2S_SCK, P2S_SDA, S2P_SCL, S2P_SDA
- net labels removed: 3VREG_SCL, 3VREG_SDA, IO12, IO23, REG_SCL, REG_SDA, RX, TX
- wire segments 134 -> 82
- no-connect marks 10 -> 12
Other:
- moved on the sheet: J122
